File: IO_NRF/IO_NRF.kicad_pcb (KiCad board)
At the start: 2 copper layers, 79 x 49.9 mm, 37 parts, among them J1 12V_IN, J2 Programmer_Pins_SPI, J3 External_Outputs_Terminal, J4 External_Inputs_Terminal, J5 XKC-Y2S-IN, K1 ST2002C12W, K2 ST2002C12W, Q1 BC817, Q2 BC817, U1 NRF24L01_Breakout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

Commit message: NRF24L01 Communicating on ESP32 & ATTINY84
IONRF + ESP32 for NRF24L01 TESTED OK.
PCBs are fixed.
Parts:
- added C7: 100nF, Capacitor_SMD:C_0603_1608Metric, F.Cu at (28.8, 37.2)
- added R12: 1k, Resistor_SMD:R_0805_2012Metric, F.Cu at (33.1, 37.2)
Connections:
- U1 pad 6: /MCU_MOSI -> /MCU_MISO
- U1 pad 7: /MCU_MISO -> /MCU_MOSI
Routing:
- net /MCU_RESET: track 34.6 -> 50.6 mm, vias 1 -> 2
- net /3V3: track 161.6 -> 153.2 mm, vias 1 -> 0
- net /MCU_MOSI: track 38.1 -> 41.3 mm, vias 3 -> 2
- net /NRF_CE: track 31.1 -> 33.7 mm, vias 0 -> 1
- net /MCU_MISO: track 49.2 -> 47.8 mm, vias 0 -> 2
- net GND: vias 32 -> 33
