File: IO_NRF/IO_NRF.kicad_sch (KiCad schematic)
At the start: 39 parts, among them J1 12V_IN, J2 Programmer_Pins_SPI, J3 External_Outputs_Terminal, J4 External_Inputs_Terminal, J5 XKC-Y2S-IN, K1 ST2002C12W, K2 ST2002C12W, Q1 BC817, Q2 BC817, U1 NRF24L01_Breakout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

Commit message: NRF24L01 Communicating on ESP32 & ATTINY84
IONRF + ESP32 for NRF24L01 TESTED OK.
PCBs are fixed.
Parts:
- added C7: 100nF, Capacitor_SMD:C_0603_1608Metric, symbol Device:C
- added R12: 1k, Resistor_SMD:R_0805_2012Metric, symbol Device:R
Connections:
- net 3V3: now also R12.1
- net GND: now also C7.1
- net MCU_MISO: now also U1.6 (MOSI); no longer U1.7 (MISO)
- net MCU_MOSI: now also U1.7 (MISO); no longer U1.6 (MOSI)
- net MCU_RESET: now also C7.2, R12.2
Changed lines of the file:
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@@
   (junction (at 176.53 39.37) (diameter 0) (color 0 0 0 0)
+  )
+  (junction (at 122.555 82.55) (diameter 0) (color 0 0 0 0)
   )
   (junction (at 73.025 118.745) (diameter 0) (color 0 0 0 0)
@@
     (stroke (width 0) (type default) (color 0 0 0 0))
   )
+  (wire (pts (xy 122.555 73.025) (xy 122.555 74.93))
+    (stroke (width 0) (type default) (color 0 0 0 0))
+  )
   (wire (pts (xy 43.815 49.53) (xy 43.815 50.8))
     (stroke (width 0) (type default) (color 0 0 0 0))
@@
   )
   (wire (pts (xy 174.625 142.875) (xy 174.625 148.59))
+    (stroke (width 0) (type default) (color 0 0 0 0))
+  )
+  (wire (pts (xy 122.555 82.55) (xy 128.27 82.55))
     (stroke (width 0) (type default) (color 0 0 0 0))
   )
@@
     (effects (font (size 1.27 1.27)) (justify left bottom))
   )
+  (label "MCU_MISO" (at 59.69 41.91 0)
+    (effects (font (size 1.27 1.27)) (justify left bottom))
+  )
   (label "RELAY_2_B_COM" (at 264.795 146.685 270)
     (effects (font (size 1.27 1.27)) (justify right bottom))
@@
     (effects (font (size 1.27 1.27)) (justify right bottom))
   )
+  (label "3V3" (at 122.555 73.025 180)
+    (effects (font (size 1.27 1.27)) (justify right bottom))
+  )
   (label "MCU_SCK" (at 59.69 36.83 0)
     (effects (font (size 1.27 1.27)) (justify left bottom))
@@
     (effects (font (size 1.27 1.27)) (justify right bottom))
   )
+  (label "MCU_MOSI" (at 59.69 39.37 0)
+    (effects (font (size 1.27 1.27)) (justify left bottom))
+  )
   (label "ACC_12V_IN" (at 182.88 128.27 180)
     (effects (font (size 1.27 1.27)) (justify right bottom))
@@
     (effects (font (size 1.27 1.27)) (justify left bottom))
   )
-  (label "MCU_MOSI" (at 59.69 41.91 0)
-    (effects (font (size 1.27 1.27)) (justify left bottom))
-  )
   (label "MCU_MOSI" (at 153.67 24.13 0)
     (effects (font (size 1.27 1.27)) (justify left bottom))
@@
     (effects (font (size 1.27 1.27)) (justify left bottom))
   )
+  (label "MCU_RESET" (at 128.27 82.55 0)
+    (effects (font (size 1.27 1.27)) (justify left bottom))
+  )
   (label "MCU_MOSI" (at 116.84 48.895 0)
     (effects (font (size 1.27 1.27)) (justify left bottom))
   )
   (label "3V3" (at 147.32 61.595 0)
-    (effects (font (size 1.27 1.27)) (justify left bottom))
-  )
-  (label "MCU_MISO" (at 59.69 39.37 0)
     (effects (font (size 1.27 1.27)) (justify left bottom))
   )
@@
     (pin "1")
   )
+  (symbol (lib_id "power:GND") (at 122.555 90.17 0) (unit 1)
+    (in_bom yes) (on_board yes) (fields_autoplaced)
+    (property "Reference" "#PWR02" (id 0) (at 122.555 96.52 0)
+      (effects (font (size 1.27 1.27)) hide)
+    )
+    (property "Value" "GND" (id 1) (at 125.095 91.4399 0)
+      (effects (font (size 1.27 1.27)) (justify left))
+    )
+    (property "Footprint" "" (id 2) (at 122.555 90.17 0)
+      (effects (font (size 1.27 1.27)) hide)
+    )
+    (property "Datasheet" "" (id 3) (at 122.555 90.17 0)
+      (effects (font (size 1.27 1.27)) hide)
+    )
+    (pin "1")
+  )
   (symbol (lib_id "power:GND") (at 182.88 162.56 0) (unit 1)
     (in_bom yes) (on_board yes) (fields_autoplaced)
@@
     (pin "2")
   )
+  (symbol (lib_id "Device:R") (at 122.555 78.74 0) (unit 1)
+    (in_bom yes) (on_board yes) (fields_autoplaced)
+    (property "Reference" "R12" (id 0) (at 125.095 77.4699 0)
+      (effects (font (size 1.27 1.27)) (justify left))
+    )
+    (property "Value" "1k" (id 1) (at 125.095 80.0099 0)
+      (effects (font (size 1.27 1.27)) (justify left))
+    )
+    (property "Footprint" "Resistor_SMD:R_0805_2012Metric" (id 2) (at 120.777 78.74 90)
+      (effects (font (size 1.27 1.27)) hide)
+    )
+    (property "Datasheet" "~" (id 3) (at 122.555 78.74 0)
+      (effects (font (size 1.27 1.27)) hide)
+    )
+    (property "Lomex" "" (id 4) (at 122.555 78.74 0)
+      (effects (font (size 1.27 1.27)) hide)
+    )
+    (property "LOMEX" "81-10-87" (id 5) (at 122.555 78.74 0)
+      (effects (font (size 1.27 1.27)) hide)
+    )
+    (pin "1")
+    (pin "2")
+  )
   (symbol (lib_id "Device:R") (at 268.605 33.02 270) (mirror x) (unit 1)
     (in_bom yes) (on_board yes) (fields_autoplaced)
@@
     )
     (pin "1")
+  )
+  (symbol (lib_id "Device:C") (at 122.555 86.36 180) (unit 1)
+    (in_bom yes) (on_board yes)
+    (property "Reference" "C7" (id 0) (at 123.825 83.82 90))
+    (property "Value" "100nF" (id 1) (at 126.365 86.36 90))
+    (property "Footprint" "Capacitor_SMD:C_0603_1608Metric" (id 2) (at 121.5898 82.55 0)
+      (effects (font (size 1.27 1.27)) hide)
+    )
+    (property "Datasheet" "~" (id 3) (at 122.555 86.36 0)
+      (effects (font (size 1.27 1.27)) hide)
+    )
+    (property "LOMEX" "82-13-28" (id 4) (at 122.555 86.36 0)
+      (effects (font (size 1.27 1.27)) hide)
+    )
+    (pin "1")
+    (pin "2")
   )
   (symbol (lib_id "power:GND") (at 98.425 74.295 0) (unit 1)
@@
       (reference "#PWR01") (unit 1) (value "GND") (footprint "")
     )
+    (path "/17c6afc7-643e-4e48-aab8-2ef6e179e245"
+      (reference "#PWR02") (unit 1) (value "GND") (footprint "")
+    )
     (path "/b1bb3d17-15dd-45c3-82fa-5de82bdfbf00"
       (reference "#PWR0101") (unit 1) (value "GND") (footprint "")
@@
       (reference "C6") (unit 1) (value "C_Polarized") (footprint "Capacitor_SMD:CP_Elec_5x5.3")
     )
+    (path "/c207590d-b044-46bd-8b35-03394f2c3802"
+      (reference "C7") (unit 1) (value "100nF") (footprint "Capacitor_SMD:C_0603_1608Metric")
+    )
     (path "/8078a9be-cd87-4f8b-9fd3-8c28a2fb1840"
       (reference "D1") (unit 1) (value "DO-214AC") (footprint "Diode_SMD:D_SMA")
@@
       (reference "R11") (unit 1) (value "1k") (footprint "Resistor_SMD:R_0805_2012Metric")
     )
+    (path "/95468fac-094d-4965-924b-3bec4290adab"
+      (reference "R12") (unit 1) (value "1k") (footprint "Resistor_SMD:R_0805_2012Metric")
+    )
     (path "/4d75bb5d-ea73-46e3-b5a8-101ec9bb8359"
