File: IO_NRF_minimal/IO_NRF_minimal.kicad_pcb (KiCad board)
At the start: 2 copper layers, 52 x 33 mm, 27 parts, among them J1 12V_IN, J2 Programmer_Pins_SPI, J3 XKC-Y2S-IN, J4 External_Inputs_Terminal, U1 NRF24L01_Breakout, U2 AP7370-33WW-7, U3 ATtiny84-20SS, U4 TLP291

Commit message: Updated both PCBs with TEMT6000 and XKC enabler
Parts:
- added JP1: SolderJumper_2_Open, Jumper:SolderJumper-2_P1.3mm_Open_RoundedPad1.0x1.5mm, B.Cu at (39.2, 37.7)
- added Q1: BC847B, Package_TO_SOT_SMD:SOT-23, F.Cu at (35.1, 33.7)
- added R3: 1k, Resistor_SMD:R_0805_2012Metric, F.Cu at (41.1, 26.8)
- moved R1 1.89 mm to (30.9, 38.2), turned to -90 degrees
Connections:
- J3 pad 2: GND -> Net-(J3-Pad2)
- U3 pad 3: unconnected-(U3-Pad3) -> /XKC_ACTIVATE
Routing:
- net Net-(J3-Pad2): track 0.00 -> 15.7 mm
- net Net-(Q1-Pad1): track 0.00 -> 10.1 mm
- net /XKC_ACTIVATE: track 0.00 -> 8.74 mm, vias 0 -> 2
- net GND: vias 27 -> 31
Other:
- board text added: "IONRF v1.2"

Commit message: Minimalized IO-NRF, no Digital Input
Parts:
- removed J4: External_Inputs_Terminal, my_kicad:SORKAPOCS-3.5mm-2
- removed R4: 1k, Resistor_SMD:R_0805_2012Metric
- removed R6: 4.7k, Resistor_SMD:R_0805_2012Metric
- removed U4: TLP291, Package_SO:SOIC-4_4.55x2.6mm_P1.27mm
Connections:
- U3 pad 13: /D_IN1 -> unconnected-(U3-Pad13)
Routing:
- net /D_IN1: track 30.0 -> 0.00 mm, vias 2 -> 0
- net Net-(R6-Pad2): track 10.8 -> 0.00 mm
- net /EXT_IN_1: track 6.20 -> 0.00 mm
- net GND: track 10.7 -> 5.69 mm, vias 31 -> 26
- net /3V3: track 99.7 -> 97.0 mm

Commit message: Updated BOMs, manufacturing (beültetés árak) and PCBs
Parts:
- C2: value 47uF -> 10uF; footprint Capacitor_SMD:CP_Elec_6.3x5.4 -> Capacitor_SMD:C_1210_3225Metric
- C6: value C_Polarized -> 100uF
- moved C2 2.16 mm to (45.4, 43.4)
Changed lines of the file:
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@@
       (effects (font (size 1 1) (thickness 0.15)))
     )
-    (fp_text value "C_Polarized" (at 0 3.7) (layer "F.Fab")
+    (fp_text value "100uF" (at 0 3.7) (layer "F.Fab")
       (effects (font (size 1 1) (thickness 0.15)))
     )
@@
     )
   )
-  (footprint "Capacitor_SMD:CP_Elec_6.3x5.4" (layer "F.Cu")
-    (at 43.7 44.75 -90)
-    (descr "SMD capacitor, aluminum electrolytic, Panasonic C55, 6.3x5.4mm")
-    (tags "capacitor electrolytic")
-    (property "LOMEX" "91-00-88 ")
-    (property "Sheetfile" "IO_NRF_minimal.kicad_sch")
-    (property "Sheetname" "")
-    (attr smd)
-    (fp_text reference "C2" (at 4.45 -2.55 180) (layer "F.SilkS")
-      (effects (font (size 1 1) (thickness 0.15)))
-    )
-    (fp_text value "47uF" (at 0 4.35 90) (layer "F.Fab")
-      (effects (font (size 1 1) (thickness 0.15)))
-    )
-    (fp_text user "${REFERENCE}" (at 0 0 90) (layer "F.Fab")
-      (effects (font (size 1 1) (thickness 0.15)))
-    )
-    (fp_line (start -4.04375 -2.24125) (end -4.04375 -1.45375) (layer "F.SilkS") (width 0.12))
-    (fp_line (start -4.4375 -1.8475) (end -3.65 -1.8475) (layer "F.SilkS") (width 0.12))
-    (fp_line (start -3.41 -2.345563) (end -2.345563 -3.41) (layer "F.SilkS") (width 0.12))
-    (fp_line (start -3.41 -2.345563) (end -3.41 -1.06) (layer "F.SilkS") (width 0.12))
-    (fp_line (start -3.41 2.345563) (end -2.345563 3.41) (layer "F.SilkS") (width 0.12))
-    (fp_line (start -2.345563 3.41) (end 3.41 3.41) (layer "F.SilkS") (width 0.12))
-    (fp_line (start 3.41 3.41) (end 3.41 1.06) (layer "F.SilkS") (width 0.12))
-    (fp_line (start -2.345563 -3.41) (end 3.41 -3.41) (layer "F.SilkS") (width 0.12))
-    (fp_line (start 3.41 -3.41) (end 3.41 -1.06) (layer "F.SilkS") (width 0.12))
-    (fp_line (start -3.41 2.345563) (end -3.41 1.06) (layer "F.SilkS") (width 0.12))
-    (fp_line (start -2.4 -3.55) (end 3.55 -3.55) (layer "F.CrtYd") (width 0.05))
-    (fp_line (start 4.8 -1.05) (end 4.8 1.05) (layer "F.CrtYd") (width 0.05))
-    (fp_line (start -3.55 -2.4) (end -3.55 -1.05) (layer "F.CrtYd") (width 0.05))
-    (fp_line (start -4.8 1.05) (end -3.55 1.05) (layer "F.CrtYd") (width 0.05))
-    (fp_line (start 3.55 -1.05) (end 4.8 -1.05) (layer "F.CrtYd") (width 0.05))
-    (fp_line (start -2.4 3.55) (end 3.55 3.55) (layer "F.CrtYd") (width 0.05))
-    (fp_line (start -3.55 -2.4) (end -2.4 -3.55) (layer "F.CrtYd") (width 0.05))
-    (fp_line (start 4.8 1.05) (end 3.55 1.05) (layer "F.CrtYd") (width 0.05))
-    (fp_line (start 3.55 1.05) (end 3.55 3.55) (layer "F.CrtYd") (width 0.05))
-    (fp_line (start -4.8 -1.05) (end -4.8 1.05) (layer "F.CrtYd") (width 0.05))
-    (fp_line (start -3.55 2.4) (end -2.4 3.55) (layer "F.CrtYd") (width 0.05))
-    (fp_line (start -3.55 1.05) (end -3.55 2.4) (layer "F.CrtYd") (width 0.05))
-    (fp_line (start -3.55 -1.05) (end -4.8 -1.05) (layer "F.CrtYd") (width 0.05))
-    (fp_line (start 3.55 -3.55) (end 3.55 -1.05) (layer "F.CrtYd") (width 0.05))
-    (fp_line (start 3.3 -3.3) (end 3.3 3.3) (layer "F.Fab") (width 0.1))
-    (fp_line (start -2.389838 -1.645) (end -2.389838 -1.015) (layer "F.Fab") (width 0.1))
-    (fp_line (start -3.3 -2.3) (end -2.3 -3.3) (layer "F.Fab") (width 0.1))
-    (fp_line (start -2.3 -3.3) (end 3.3 -3.3) (layer "F.Fab") (width 0.1))
-    (fp_line (start -3.3 2.3) (end -2.3 3.3) (layer "F.Fab") (width 0.1))
-    (fp_line (start -3.3 -2.3) (end -3.3 2.3) (layer "F.Fab") (width 0.1))
-    (fp_line (start -2.3 3.3) (end 3.3 3.3) (layer "F.Fab") (width 0.1))
-    (fp_line (start -2.704838 -1.33) (end -2.074838 -1.33) (layer "F.Fab") (width 0.1))
-    (fp_circle (center 0 0) (end 3.15 0) (layer "F.Fab") (width 0.1) (fill none))
-    (pad "1" smd roundrect (at -2.8 0 270) (size 3.5 1.6) (layers "F.Cu" "F.Paste" "F.Mask") (roundrect_rratio 0.15625)
-      (net 3 "/3V3") (pintype "passive"))
-    (pad "2" smd roundrect (at 2.8 0 270) (size 3.5 1.6) (layers "F.Cu" "F.Paste" "F.Mask") (roundrect_rratio 0.15625)
+  (footprint "Capacitor_SMD:C_1210_3225Metric" (layer "F.Cu")
+    (at 45.39 43.4 -90)
+    (descr "Capacitor SMD 1210 (3225 Metric), square (rectangular) end terminal, IPC_7351 nominal, (Body size source: IPC-SM-782 page 76, https://www.pcb-3d.com/wordpress/wp-content/uploads/ipc-sm-782a_amendment_1_and_2.pdf), generated with kicad-footprint-generator")
+    (tags "capacitor")
+    (property "LOMEX" "82-08-34")
+    (property "Sheetfile" "IO_NRF_minimal.kicad_sch")
+    (property "Sheetname" "")
+    (attr smd)
+    (fp_text reference "C2" (at -3.03 -0.05) (layer "F.SilkS")
+      (effects (font (size 1 1) (thickness 0.15)))
+    )
+    (fp_text value "10uF" (at 0 2.3 -90) (layer "F.Fab")
+      (effects (font (size 1 1) (thickness 0.15)))
+    )
+    (fp_text user "${REFERENCE}" (at 0 0 -90) (layer "F.Fab")
+      (effects (font (size 0.8 0.8) (thickness 0.12)))
+    )
+    (fp_line (start -0.711252 -1.36) (end 0.711252 -1.36) (layer "F.SilkS") (width 0.12))
+    (fp_line (start -0.711252 1.36) (end 0.711252 1.36) (layer "F.SilkS") (width 0.12))
+    (fp_line (start 2.3 1.6) (end -2.3 1.6) (layer "F.CrtYd") (width 0.05))
+    (fp_line (start -2.3 1.6) (end -2.3 -1.6) (layer "F.CrtYd") (width 0.05))
+    (fp_line (start 2.3 -1.6) (end 2.3 1.6) (layer "F.CrtYd") (width 0.05))
+    (fp_line (start -2.3 -1.6) (end 2.3 -1.6) (layer "F.CrtYd") (width 0.05))
+    (fp_line (start -1.6 -1.25) (end 1.6 -1.25) (layer "F.Fab") (width 0.1))
+    (fp_line (start 1.6 1.25) (end -1.6 1.25) (layer "F.Fab") (width 0.1))
+    (fp_line (start 1.6 -1.25) (end 1.6 1.25) (layer "F.Fab") (width 0.1))
+    (fp_line (start -1.6 1.25) (end -1.6 -1.25) (layer "F.Fab") (width 0.1))
+    (pad "1" smd roundrect (at -1.475 0 270) (size 1.15 2.7) (layers "F.Cu" "F.Paste" "F.Mask") (roundrect_rratio 0.217391)
+      (net 3 "/3V3") (pintype "passive"))
+    (pad "2" smd roundrect (at 1.475 0 270) (size 1.15 2.7) (layers "F.Cu" "F.Paste" "F.Mask") (roundrect_rratio 0.217391)
       (net 2 "GND") (pintype "passive"))
-    (model "${KICAD6_3DMODEL_DIR}/Capacitor_SMD.3dshapes/CP_Elec_6.3x5.4.wrl"
-      (offset (xyz 0 0 0))
-      (scale (xyz 1 1 1))
+    (model "${KICAD6_3DMODEL_DIR}/Capacitor_SMD.3dshapes/C_1210_3225Metric.wrl"
+      (offset (xyz 0 0 0))
+      (scale (xyz 1 1 1))

Commit message: latest versions
Parts:
- U1: value NRF24L01_Breakout -> NRF24L01_SMD
Connections:
- U1 pad 1: GND -> /3V3
- U1 pad 2: /3V3 -> GND
- U1 pad 9: (no net) -> unconnected-(U1-Pad9)
Routing:
- net /3V3: track 97.0 -> 96.5 mm
Other:
- board text added: "IONRF v1.21"
- board text removed: "IONRF v1.2"
